Commit message: Imported upstream version '0.0.5' of 'upstream'

File: multi_jackal_description/urdf/accessories/twocams.urdf.xacro (robot description, xacro)
@@ -2,5 +2,5 @@
 <robot >
   <!-- Front camera. -->
-  <joint name="front_camera_mount_joint" type="fixed">
+  <!--<joint name="front_camera_mount_joint" type="fixed">
     <origin xyz="0.060 0 0" rpy="0 0 0" />
     <parent link="front_mount" />
@@ -18,9 +18,8 @@
                           camera_mass="0.085" hfov="1.0471975512" fps="60" width="640" height="512"/>
   <joint name="front_camera_bracket_joint" type="fixed">
-    <!-- Alter tilt here or set FLEAR3_CAMERA_TILT var. Default was 0.5236. -->
     <origin xyz="0.030 0 0.008" rpy="0 $(optenv FLEA3_CAMERA_TILT 0) 0" />
     <parent link="front_camera_pivot" />
     <child link="front_camera" />
-  </joint>
+  </joint>-->
   <!-- Rear camera. INCOMPLETE, NO IMAGE CREATED.-->
   <joint name="rear_camera_mount_joint" type="fixed">

File: multi_jackal_description/urdf/base_accessories.urdf.xacro (robot description, xacro)
@@ -34,5 +34,5 @@
   <xacro:if value="$(optenv JACKAL_FLEA3 0)">
     <camera_mount prefix="$(optenv JACKAL_FLEA_MOUNT front)"
-                       tilt="$(optenv JACKAL_FLEA_TILT 0.5236)"/>
+                       tilt="$(optenv JACKAL_FLEA_TILT 0)"/>
     <joint name="$(optenv JACKAL_FLEA3_MOUNT front)_camera_mount_joint" type="fixed">
       <origin xyz="$(optenv JACKAL_FLEA3_OFFSET 0 0 0)"

File: multi_jackal_description/urdf/custom_accessories.urdf.xacro (robot description, xacro)
@@ -18,3 +18,7 @@
     <xacro:include filename="accessories/twocams.urdf.xacro"/>
   </xacro:if>
+  <!-- Box with AprilTag markers on each face, lifted up slightly. -->
+  <xacro:if value="$(optenv JACKAL_APRILTAG_POLE 0)">
+    <xacro:include filename="accessories/apriltag_box_with_pole.urdf.xacro" />
+  </xacro:if>
 </robot>
